File: SCH_PCB/LEDBOARD01A/LEDBOARD01A.sch (KiCad schematic (older format))
At the start: 11 parts, among them J1 JUMP_3X2, J2 CONN_2, P1 USB_B, U1 MPC1643

Commit message: Modifications
Parts:
- U1: value MPC1643 -> MCP1643
Changed lines of the file:
@@
 P 6350 3050
 F 0 "U1" H 6500 3600 60  0000 C CNN
-F 1 "MPC1643" H 6350 3050 60  0000 C CNN
+F 1 "MCP1643" H 6350 3050 60  0000 C CNN
 F 2 "Mlab_IO:MSOP-8_3x3mm_Pitch0.65mm" H 6350 3050 60  0001 C CNN
 F 3 "" H 6350 3050 60  0000 C CNN
@@
 Connection ~ 4450 2250
 Connection ~ 6950 3250
-Connection ~ 6000 4800
 $Comp
 L LED D2
