File: SCH_PCB/LEDBOARD01A/LEDBOARD01A.kicad_pcb (KiCad board)
At the start: 2 copper layers, 30 x 20 mm, 11 parts, among them J1 JUMP_3X2, J2 CONN_2, P1 USB_B, U1 MPC1643

Commit message: Modifications
Parts:
- U1: value MPC1643 -> MCP1643
Other:
- rule pad_to_mask_clearance: 0.2 -> 0.1
- rule via_min_size: 0.4 -> 0.7
Changed lines of the file:
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@@
     (links 32)
     (no_connects 0)
-    (area -0.100001 -20.100001 30.100001 0.100001)
+    (area -2.032 -21.701571 31.8992 1.524001)
     (thickness 1.6)
     (drawings 6)
@@
     (via_size 0.8)
     (via_drill 0.4)
-    (via_min_size 0.4)
+    (via_min_size 0.7)
     (via_min_drill 0.3)
     (uvia_size 0.3)
     (uvia_drill 0.1)
     (uvias_allowed no)
-    (uvia_min_size 0.2)
+    (uvia_min_size 0.3)
     (uvia_min_drill 0.1)
     (pcb_text_width 0.3)
@@
     (pad_size 1.524 1.524)
     (pad_drill 0.762)
-    (pad_to_mask_clearance 0.2)
+    (pad_to_mask_clearance 0.1)
     (aux_axis_origin 0 0)
     (visible_elements 7FFFFF7F)
     (pcbplotparams
-      (layerselection 0x00030_80000001)
+      (layerselection 0x010e0_80000001)
       (usegerberextensions false)
       (excludeedgelayer true)
@@
       (outputformat 1)
       (mirror false)
-      (drillshape 1)
+      (drillshape 0)
       (scaleselection 1)
-      (outputdirectory ""))
+      (outputdirectory CAM_PROFI/))
   )
   (net 0 "")
@@
       (effects (font (size 1 1) (thickness 0.15)) (justify mirror))
     )
-    (fp_text value MPC1643 (at 0 -2.6 180) (layer B.SilkS)
+    (fp_text value MCP1643 (at 0 -2.6 180) (layer B.SilkS)
       (effects (font (size 1 1) (thickness 0.15)) (justify mirror))
     )
