File: SCH_PCB/CAPLIGHT01A/CAPLIGHT01A.sch (KiCad schematic (older format))
At the start: 16 parts, among them J1 JUMP_3X2, J2 CONN1_1, J3 JUMP_2x1, P1 USB_OTG, U1 LTC3625

Commit message: New charge indicating LED added. Manufacturing files generated.
Parts:
- removed J2: CONN1_1, Measurement_Points:Measurement_Point_Round-SMD-Pad_Small, symbol CONN1_1
- removed J3: JUMP_2x1, Measurement_Points:Measurement_Point_Round-SMD-Pad_Small, symbol JUMP_2x1
- removed R2: 287k, Mlab_R:SMD-0805, symbol R
- removed R3: 100k, Mlab_R:SMD-0805, symbol R
- added D3: LED, Mlab_D:LED_1206, symbol LED
- added R6: 1k, Mlab_R:SMD-0805, symbol R
- C3: value 22F -> 50F
- R1: value - -> 0
- R5: value ??k -> 1k; footprint Mlab_R:SMD-0805 -> Mlab_R:SMD-1206
Connections:
- net EN is gone; now on net VIN: U1.5 (EN)
- net PG: now also D3.1 (K)
- net VIN: now also U1.7 (PFI), R6.1
- net #PFO: no longer names the net of U1.8 (PFO)
- new net: D3.2 (A), R6.2
Changed lines of the file:
@@
 EESchema Schematic File Version 2
-LIBS:MLAB_BATERY
-LIBS:MLAB_CONNECTORS
-LIBS:MLAB_D
-LIBS:MLAB_HEADER
-LIBS:MLAB_IO
-LIBS:MLAB_Jumpers
-LIBS:MLAB_MECHANICAL
-LIBS:MLAB_SW
-LIBS:MLAB_T
-LIBS:MLAB_U
 LIBS:power
 LIBS:device
@@
 P 7850 3550
 F 0 "C3" H 7875 3650 50  0000 L CNN
-F 1 "22F" H 7875 3450 50  0000 L CNN
+F 1 "50F" H 7875 3450 50  0000 L CNN
 F 2 "Mlab_C:C_Radial_D18_L25_P7.5" H 7888 3400 50  0001 C CNN
 F 3 "" H 7850 3550 50  0000 C CNN
@@
 	1    0    0    -1
 $EndComp
-$Comp
-L CONN1_1 J2
-U 1 1 56E82602
-P 5000 3300
-F 0 "J2" H 5050 3350 50  0000 C CNN
-F 1 "CONN1_1" H 5100 3250 40  0001 C CNN
-F 2 "Measurement_Points:Measurement_Point_Round-SMD-Pad_Small" H 5050 3250 60  0001 C CNN
-F 3 "" H 5050 3250 60  0000 C CNN
-	1    5000 3300
-	-1   0    0    1
-$EndComp
-Wire Wire Line
-	5850 3350 5300 3350
+Wire Wire Line
+	4850 3350 5850 3350
 Wire Wire Line
 	5850 2900 3700 2900
@@
 $EndComp
 Connection ~ 4850 2900
-Text Label 5300 3350 0    60   ~ 0
-EN
 Text Label 3900 2900 0    60   ~ 0
 VIN
-$Comp
-L R R3
-U 1 1 56E84F85
-P 5750 4300
-F 0 "R3" H 5681 4346 50  0000 R CNN
-F 1 "100k" H 5681 4255 50  0000 R CNN
-F 2 "Mlab_R:SMD-0805" V 5680 4300 50  0001 C CNN
-F 3 "" H 5750 4300 50  0000 C CNN
-	1    5750 4300
-	1    0    0    -1
-$EndComp
-$Comp
-L R R2
-U 1 1 56E85082
-P 5750 3900
-F 0 "R2" V 5830 3900 50  0000 C CNN
-F 1 "287k" V 5750 3900 50  0000 C CNN
-F 2 "Mlab_R:SMD-0805" V 5680 3900 50  0001 C CNN
-F 3 "" H 5750 3900 50  0000 C CNN
-	1    5750 3900
-	1    0    0    -1
-$EndComp
-Wire Wire Line
-	5750 3750 5750 3650
-Text Label 5750 3650 0    60   ~ 0
-VIN
-$Comp
-L GND #PWR04
-U 1 1 56E85820
-P 5750 4500
-F 0 "#PWR04" H 5750 4250 50  0001 C CNN
-F 1 "GND" H 5750 4350 50  0000 C CNN
-F 2 "" H 5750 4500 50  0000 C CNN
-F 3 "" H 5750 4500 50  0000 C CNN
-	1    5750 4500
-	1    0    0    -1
-$EndComp
-Wire Wire Line
-	5750 4500 5750 4450
-Wire Wire Line
-	5750 4150 5750 4050
-Wire Wire Line
-	5850 4100 5750 4100
-Connection ~ 5750 4100
 $Comp
 L R R4
@@
 	6150 4850 6150 4800
 $Comp
-L GND #PWR05
+L GND #PWR04
 U 1 1 56E8600D
 P 6150 5200
-F 0 "#PWR05" H 6150 4950 50  0001 C CNN
+F 0 "#PWR04" H 6150 4950 50  0001 C CNN
 F 1 "GND" H 6150 5050 50  0000 C CNN
 F 2 "" H 6150 5200 50  0000 C CNN
@@
 	6150 5200 6150 5150
 $Comp
-L GND #PWR06
+L GND #PWR05
 U 1 1 56E86076
 P 6400 4850
-F 0 "#PWR06" H 6400 4600 50  0001 C CNN
+F 0 "#PWR05" H 6400 4600 50  0001 C CNN
 F 1 "GND" H 6400 4700 50  0000 C CNN
 F 2 "" H 6400 4850 50  0000 C CNN
@@
 Wire Wire Line
 	7700 3700 6800 3700
-Wire Wire Line
-	6800 4100 7050 4100
-Text Label 6800 4100 0    60   ~ 0
-#PFO
 Text Label 6800 4250 0    60   ~ 0
 PG
@@
 	3850 2400 3900 2400
 $Comp
-L GND #PWR07
+L GND #PWR06
 U 1 1 5771AF62
 P 4050 2100
-F 0 "#PWR07" H 4050 1850 50  0001 C CNN
+F 0 "#PWR06" H 4050 1850 50  0001 C CNN
 F 1 "GND" H 4055 1927 50  0000 C CNN
 F 2 "" H 4050 2100 50  0000 C CNN
@@
 P 8350 3550
 F 0 "R5" V 8430 3550 50  0000 C CNN
-F 1 "??k" V 8350 3550 50  0000 C CNN
-F 2 "Mlab_R:SMD-0805" V 8280 3550 50  0001 C CNN
+F 1 "1k" V 8350 3550 50  0000 C CNN
+F 2 "Mlab_R:SMD-1206" V 8280 3550 50  0001 C CNN
 F 3 "" H 8350 3550 50  0000 C CNN
 	1    8350 3550
@@
 $EndComp
 $Comp
-L GND #PWR08
+L GND #PWR07
 U 1 1 57728495
 P 7850 3800
-F 0 "#PWR08" H 7850 3550 50  0001 C CNN
+F 0 "#PWR07" H 7850 3550 50  0001 C CNN
 F 1 "GND" H 7855 3627 50  0000 C CNN
 F 2 "" H 7850 3800 50  0000 C CNN
@@
 	7850 3800 7850 3700
 $Comp
-L GND #PWR09
+L GND #PWR08
 U 1 1 5776E87A
 P 8350 4100
-F 0 "#PWR09" H 8350 3850 50  0001 C CNN
+F 0 "#PWR08" H 8350 3850 50  0001 C CNN
 F 1 "GND" H 8355 3927 50  0000 C CNN
 F 2 "" H 8350 4100 50  0000 C CNN
@@
 P 5650 3150
 F 0 "R1" V 5730 3150 50  0000 C CNN
-F 1 "-" V 5650 3150 50  0000 C CNN
+F 1 "0" V 5650 3150 50  0000 C CNN
 F 2 "Mlab_R:SMD-0805" V 5580 3150 50  0001 C CNN
 F 3 "" H 5650 3150 50  0000 C CNN
@@
 	8350 3350 8350 3400
 Wire Wire Line
-	4850 3550 4850 2900
+	4850 2900 4850 4100
 Wire Wire Line
 	6800 3550 6800 3250
 Connection ~ 6800 3250
-$Comp
-L JUMP_2x1 J3
-U 1 1 57791ABD
-P 7450 4250
-F 0 "J3" H 7100 4450 50  0000 C CNN
-F 1 "JUMP_2x1" V 7450 4400 40  0001 C CNN
-F 2 "Measurement_Points:Measurement_Point_Round-SMD-Pad_Small" H 7450 4250 60  0001 C CNN
-F 3 "" H 7450 4250 60  0000 C CNN
-	1    7450 4250
-	1    0    0    -1
-$EndComp
 Wire Wire Line
 	7850 2900 6800 2900
+Connection ~ 4850 3550
+$Comp
+L R R6
+U 1 1 577C016E
+P 7700 4550
+F 0 "R6" V 7780 4550 50  0000 C CNN
+F 1 "1k" V 7700 4550 50  0000 C CNN
+F 2 "Mlab_R:SMD-0805" V 7630 4550 50  0001 C CNN
+F 3 "" H 7700 4550 50  0000 C CNN
+	1    7700 4550
+	1    0    0    -1
+$EndComp
+$Comp
+L LED D3
+U 1 1 577C0351
+P 7700 4950
+F 0 "D3" V 7746 4842 50  0000 R CNN
+F 1 "LED" V 7655 4842 50  0000 R CNN
+F 2 "Mlab_D:LED_1206" H 7700 4950 50  0001 C CNN
+F 3 "" H 7700 4950 50  0000 C CNN
+	1    7700 4950
+	0    -1   -1   0
+$EndComp
+Wire Wire Line
+	7700 4400 7700 4250
+Wire Wire Line
+	7700 4700 7700 4750
+Wire Wire Line
+	7700 5150 7700 5300
+Wire Wire Line
+	7700 5300 6950 5300
+Wire Wire Line
+	6950 5300 6950 4250
+Wire Wire Line
+	6950 4250 6800 4250
+Text Label 7700 4250 0    60   ~ 0
+VIN
+Wire Wire Line
+	4850 4100 5850 4100
+Connection ~ 4850 3350
 $EndSCHEMATC

Commit message: Components values in schema changed to real values populated on PCBs. A photo added to the readme file.
Parts:
- R4: value 71.5k -> 133k
- R5: value 1k -> 68
- R6: value 1k -> 270
Changed lines of the file:
@@
 P 6150 5000
 F 0 "R4" V 6230 5000 50  0000 C CNN
-F 1 "71.5k" V 6150 5000 50  0000 C CNN
+F 1 "133k" V 6150 5000 50  0000 C CNN
 F 2 "Mlab_R:SMD-0805" V 6080 5000 50  0001 C CNN
 F 3 "" H 6150 5000 50  0000 C CNN
@@
 P 8350 3550
 F 0 "R5" V 8430 3550 50  0000 C CNN
-F 1 "1k" V 8350 3550 50  0000 C CNN
+F 1 "68" V 8350 3550 50  0000 C CNN
 F 2 "Mlab_R:SMD-1206" V 8280 3550 50  0001 C CNN
 F 3 "" H 8350 3550 50  0000 C CNN
@@
 P 7700 4550
 F 0 "R6" V 7780 4550 50  0000 C CNN
-F 1 "1k" V 7700 4550 50  0000 C CNN
+F 1 "270" V 7700 4550 50  0000 C CNN
 F 2 "Mlab_R:SMD-0805" V 7630 4550 50  0001 C CNN
 F 3 "" H 7700 4550 50  0000 C CNN
