File: SCH_PCB/CAPLIGHT01B/CAPLIGHT01B.sch (KiCad schematic (older format))
At the start: 14 parts, among them J1 JUMP_3X2, P1 USB_OTG, U1 LTC3625

Commit message: Opravy výrobní data
Generována nová data. Zvětšen otvor pro C 50F.
Parts:
- C3: footprint Mlab_C:C_Radial_D18_L25_P7.5 -> Mlab_C:C_Radial_D18_L25_P7.5_BAT
Changed lines of the file:
@@
 LIBS:adc-dac
 LIBS:memory
-LIBS:xilinx
 LIBS:microcontrollers
 LIBS:dsp
@@
 LIBS:contrib
 LIBS:valves
-LIBS:CAPLIGHT01A-cache
+LIBS:CAPLIGHT01B-cache
 EELAYER 25 0
 EELAYER END
@@
 F 0 "C3" H 7875 3650 50  0000 L CNN
 F 1 "50F" H 7875 3450 50  0000 L CNN
-F 2 "Mlab_C:C_Radial_D18_L25_P7.5" H 7888 3400 50  0001 C CNN
+F 2 "Mlab_C:C_Radial_D18_L25_P7.5_BAT" H 7888 3400 50  0001 C CNN
 F 3 "" H 7850 3550 50  0000 C CNN
 	1    7850 3550
