File: SCH_PCB/CAPLIGHT01B/CAPLIGHT01B.sch (KiCad schematic (older format))
At the start: 14 parts, among them J1 JUMP_3X2, P1 MX-105017-0001, U1 LTC3625

Commit message: Documentation updated, english texts improved. Idicator LED changed to green in schematics.
Parts:
- D2: symbol LED -> LED-RESCUE-CAPLIGHT01B
- D3: value RED -> GREEN; symbol LED -> LED-RESCUE-CAPLIGHT01B
- P1: symbol USB_OTG -> USB_OTG-RESCUE-CAPLIGHT01B
Changed lines of the file:
@@
 EESchema Schematic File Version 2
+LIBS:CAPLIGHT01B-rescue
 LIBS:power
 LIBS:device
@@
 LIBS:adc-dac
 LIBS:memory
+LIBS:xilinx
 LIBS:microcontrollers
 LIBS:dsp
@@
 LIBS:valves
 LIBS:CAPLIGHT01B-cache
-EELAYER 25 0
+EELAYER 26 0
 EELAYER END
 $Descr A4 11693 8268
@@
 	3900 2400 3900 2950
 $Comp
-L USB_OTG P1
+L USB_OTG-RESCUE-CAPLIGHT01B P1
 U 1 1 5771AC18
 P 3550 2200
@@
 Connection ~ 4050 2000
 $Comp
-L LED D2
+L LED-RESCUE-CAPLIGHT01B D2
 U 1 1 5771A40B
 P 8350 3900
@@
 $EndComp
 $Comp
-L LED D3
+L LED-RESCUE-CAPLIGHT01B D3
 U 1 1 577C0351
 P 7700 4950
 F 0 "D3" V 7746 4842 50  0000 R CNN
-F 1 "RED" V 7655 4842 50  0000 R CNN
+F 1 "GREEN" V 7655 4842 50  0000 R CNN
 F 2 "Mlab_D:LED_1206" H 7700 4950 50  0001 C CNN
 F 3 "" H 7700 4950 50  0000 C CNN
